File: Hardware/brd_final.brd (EAGLE design)
At the start: 170.2 x 111.2 mm, 103 parts, among them IC1 XC6220A331MR-G, IC2 BD5229G-TR, J1 FH34SRJ-24S-0.5SH_99_, J2 SAMACSYS_PARTS_USB4110-GF-A, J3 QWIIC_RIGHT_ANGLE, J4 112A-TAAR-R03_ATTEND, Q1 20V/4.2A/52mΩ/1.4W, Q2 20V/4.2A/52mΩ/1.4W, Q4 SI1308EDL-T1-GE3, U1 ESP32-C6-WROOM-1-N8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

Commit message: final
final
Parts:
- 3V3, EPD_3V3, EPD_3V3_C, EPD_BUSY, EPD_CS, EPD_DC, EPD_RST, GND_1, GND_2, INT_RTC, MISO, MOSI, RX, SCK, TX, VBAT, VBUS: value TPTP20R -> TP
- D10, D11, D6, D7, D8, D9: value PGB1010603MR -> PGB1010603MRCEVA2
- D3, D4, D5: value MBR0530 -> MBR0530CEVA
Connections:
- net 12C_PW renamed I2C_PW
Routing:
- net SRC: track 39.9 -> 42.8 mm
- net GND: vias 7 -> 36
