File: Hardware/schema_final.sch (EAGLE design)
At the start: 103 parts, among them IC1 XC6220A331MR-G, IC2 BD5229G-TR, J1 FH34SRJ-24S-0.5SH_99_, J2 SAMACSYS_PARTS_USB4110-GF-A, J3 QWIIC_RIGHT_ANGLE, J4 112A-TAAR-R03_ATTEND, Q1 20V/4.2A/52mΩ/1.4W, Q2 20V/4.2A/52mΩ/1.4W, Q4 SI1308EDL-T1-GE3, U1 ESP32-C6-WROOM-1-N8, U2 W25Q512JVEIQ, U3 DS3231SN#, U4 MAX17048G+T10

Commit message: final
final
Parts:
- 3V3, EPD_3V3, EPD_3V3_C, EPD_BUSY, EPD_CS, EPD_DC, EPD_RST, GND_1, GND_2, INT_RTC, MISO, MOSI, RX, SCK, TX, VBAT, VBUS: value TPTP20R -> TP; device DeskAssistant v19 v1:TPTP20R -> DeskAssistant v19 v1:TP
- C1, C10, C1_BAT, C1_BAT1, C1_BAT2, C1_SENS, C2_BAT, C2_SENS, C4, C4_USB, C5, C5_USB, C6, C7, C9, C_DELAY, EPD_C1, EPD_C10, EPD_C11, EPD_C12, EPD_C2, EPD_C5, EPD_C6, EPD_C7, EPD_C8, EPD_C9: device DeskAssistant v19 v1:EAGLE-LTSPICE_CC0402 -> DeskAssistant v19 v1:EAGLE-LTSPICE_C
- D10, D11, D6, D7, D8, D9: value PGB1010603MR -> PGB1010603MRCEVA2; device DeskAssistant v19 v1:PGB1010603MR -> DeskAssistant v19 v1:PGB1010603MRCEVA2
- D3, D4, D5: value MBR0530 -> MBR0530CEVA; device DeskAssistant v19 v1:MBR0530 -> DeskAssistant v19 v1:MBR0530CEVA
- Q1, Q2: device DeskAssistant v19 v1:ESP32_WROVER_SPARKFUN-DISCRETESEMI_MOSFET_PCH-DMG2305UX-7 -> DeskAssistant v19 v1:ESP32_WROVER_SPARKFUN-DISCRETESEMI_MOSFET_PCH; PROD_ID DMG2305UX-7 -> (none)
- R1, R10, R12, R13, R1_BAT, R1_PINH, R1_PWRUSB, R2, R2-USB1, R2-USB2, R2_BAT, R2_PINH, R3, R4, R5, R6, R7, R8, R9, R_BOOT, R_CAPACITOR, R_CHANGE, R_CL1, R_RESET: device DeskAssistant v19 v1:ESP32_WROVER_EAGLE-LTSPICE_RR0402 -> DeskAssistant v19 v1:ESP32_WROVER_EAGLE-LTSPICE_R
Connections:
- net 12C_PW renamed I2C_PW
